File: Project Files/PCB Layouts/AutoSpiel/AutoSpielSimplified.brd (EAGLE design)
At the start: 264.1 x 83.5 mm, 134 parts, among them X1 5566-24

Commit message: Created 2 versions of the finished board
Parts:
- moved NU32_JACK 407.9 mm to (273.1, 63.5)
- moved QF#3 255.6 mm to (111.8, 105.4), turned to 270 degrees
- moved QG3 235.3 mm to (118.1, 113.0), turned to 270 degrees
- moved QG#3 208.3 mm to (124.5, 113.0), turned to 270 degrees
- moved NU32RIGHT 2.54 mm to (261.6, 68.6)
- moved NYU32LEFT 2.54 mm to (243.8, 68.6)
Other:
- board size 264.1 x 83.5 mm -> 283.2 x 83.5 mm
