File: Project Files/PCB Layouts/AutoSpiel/AutoSpielSimplified 2 Finished.brd (EAGLE design)
At the start: 266.7 x 91.1 mm, 134 parts, among them X1 5566-24

Commit message: Labeled everything on the board layout
Routing:
- net VDD2: track 347.6 -> 510.9 mm, vias 0 -> 2
- net VDD1: track 244.4 -> 371.8 mm
- net A3: track 165.1 -> 271.1 mm, vias 2 -> 4
- net A#4: track 113.4 -> 209.9 mm, vias 3 -> 10
- net F2: track 265.8 -> 351.8 mm, vias 4 -> 6
- net B3: track 162.0 -> 245.2 mm, vias 2 -> 5
- net G2: track 256.7 -> 317.5 mm, vias 6 -> 9
- net E4: track 210.0 -> 156.8 mm
- net G#2: track 217.7 -> 265.6 mm, vias 2 -> 3
- net NU32GND: track 305.0 -> 261.8 mm
- net N$14: track 92.3 -> 51.1 mm
- net C3: track 196.4 -> 235.7 mm, vias 2 -> 5
- net G4: track 171.8 -> 132.6 mm
- net D3: track 185.2 -> 218.5 mm, vias 2 -> 9
- net B2: track 203.3 -> 235.3 mm, vias 2 -> 5
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Other:
- board size 266.7 x 91.1 mm -> 270.5 x 91.1 mm
- board text added: "A#2"
- board text added: "A#3"
- board text added: "A#4"
- board text added: "A2"
- board text added: "A3"
- board text added: "A4"
- board text added: "AUTOSPIEL v1.0a"
- board text added: "B2"
- board text added: "B3"
- board text added: "B4"
- board text added: "C#3"
- board text added: "C#4"
- board text added: "C3"
- board text added: "C4"
- board text added: "C5"
- board text added: "D#3"
- board text added: "D#4"
- board text added: "D3"
- board text added: "D4"
- board text added: "Designer: Jonathan Westerfield '19"
- board text added: "E3"
- board text added: "E4"
- board text added: "F#2"
- board text added: "F#3"
- board text added: "F#4"
- board text added: "F2"
- board text added: "F3"
- board text added: "F4"
- board text added: "G#2"
- board text added: "G#3"
- board text added: "G#4"
- board text added: "G2"
- board text added: "G3"
- board text added: "G4"
- board text added: "NU_32 PWR"
- board text added: "OFF"
- board text added: "ON"
- board text added: "PSU PWR CONN"
- board text added: "RPI PWR"
