File: Project Files/PCB Layouts/AutoSpiel/AutoSpielSimplified 3 Finished.brd (EAGLE design)
At the start: 266.7 x 91.1 mm, 134 parts, among them X1 5566-24

Commit message: Added labels on the board
Other:
- board size 266.7 x 91.1 mm -> 271.8 x 91.1 mm
- board text added: "A#2"
- board text added: "A#3"
- board text added: "A#4"
- board text added: "A2"
- board text added: "A3"
- board text added: "A4"
- board text added: "AUTOSPIEL v1.0b"
- board text added: "B2"
- board text added: "B3"
- board text added: "B4"
- board text added: "C#3"
- board text added: "C#4"
- board text added: "C3"
- board text added: "C4"
- board text added: "C5"
- board text added: "D#3"
- board text added: "D#4"
- board text added: "D3"
- board text added: "D4"
- board text added: "Designer: Jonathan Westerfield '19"
- board text added: "E3"
- board text added: "E4"
- board text added: "F#2"
- board text added: "F#3"
- board text added: "F#4"
- board text added: "F2"
- board text added: "F3"
- board text added: "F4"
- board text added: "G#2"
- board text added: "G#3"
- board text added: "G#4"
- board text added: "G2"
- board text added: "G3"
- board text added: "G4"
- board text added: "NU32_PWR"
- board text added: "OFF"
- board text added: "ON"
- board text added: "PSU_PWR_CONN"
- board text added: "RPI_PWR"
