File: Project Files/PCB Layouts/AutoSpiel/AutoSpiel v1.2a.brd (EAGLE design)
At the start: 270.5 x 94.9 mm, 134 parts, among them X1 5566-24

Commit message: Finished and finalized Autospiel v1.3a. Created gerber files but need to confirm they are correct
Routing:
- net VDD2: track 0.00 -> 349.1 mm
- net NU32GND: track 0.00 -> 307.0 mm
- net F#2: track 0.00 -> 286.5 mm, vias 0 -> 3
- net NU32PWR: track 0.00 -> 272.1 mm, vias 0 -> 2
- net G#2: track 0.00 -> 264.2 mm, vias 0 -> 3
- net A#3: track 0.00 -> 255.2 mm, vias 0 -> 6
- net A3: track 0.00 -> 245.5 mm, vias 0 -> 4
- net VDD1: track 0.00 -> 244.1 mm
- net B3: track 0.00 -> 243.2 mm, vias 0 -> 6
- net RPI_GND: track 0.00 -> 238.1 mm
- net F2: track 0.00 -> 236.2 mm, vias 0 -> 3
- net RPI_PWR: track 0.00 -> 231.7 mm
- net G2: track 0.00 -> 229.3 mm, vias 0 -> 3
- net C4: track 0.00 -> 225.1 mm, vias 0 -> 6
- net A2: track 0.00 -> 213.2 mm, vias 0 -> 2
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Other:
- board text added: "AUTOSPIEL v1.2a GND Layer"
- board text removed: "AUTOSPIEL v1.1a GND Layer"
